Commit message: update ROS2 version

File: urdf/ai_car.urdf (robot description, URDF)
Before this commit: robot ai_car, 11 links, 10 joints
Links:
- link arm_link_1: geometry collision mesh filename=package://ai_car/meshes/arm_link_1.stl scale=0.001 0.001 0.001; visual mesh filename=package://ai_car/meshes/arm_link_1.stl scale=0.001 0.001 0.001
- link arm_link_2: geometry collision mesh filename=package://ai_car/meshes/arm_link_2.stl scale=0.001 0.001 0.001; visual mesh filename=package://ai_car/meshes/arm_link_2.stl scale=0.001 0.001 0.001
- link arm_tool: geometry collision mesh filename=package://ai_car/meshes/arm_tool.stl scale=0.001 0.001 0.001; visual mesh filename=package://ai_car/meshes/arm_tool.stl scale=0.001 0.001 0.001
- link base_link: geometry collision box size=0.27 0.14 0.19; visual mesh filename=package://ai_car/meshes/base_link.stl scale=0.001 0.001 0.001
- link base_scan: geometry collision cylinder length=0.0315 radius=0.055; visual mesh filename=package://ai_car/meshes/RP-lidar-A1.stl scale=0.001 0.001 0.001
- link wheel_left_link: geometry collision cylinder length=0.018 radius=0.033; visual mesh filename=package://ai_car/meshes/left_tire.stl scale=0.001 0.001 0.001
- link wheel_rear_left_link: geometry collision cylinder length=0.018 radius=0.033; visual mesh filename=package://ai_car/meshes/left_tire.stl scale=0.001 0.001 0.001
- link wheel_rear_right_link: geometry collision cylinder length=0.018 radius=0.033; visual mesh filename=package://ai_car/meshes/right_tire.stl scale=0.001 0.001 0.001
- link wheel_right_link: geometry collision cylinder length=0.018 radius=0.033; visual mesh filename=package://ai_car/meshes/right_tire.stl scale=0.001 0.001 0.001
Joints:
- joint arm_joint_1: axis 0 1 0 -> 0 -1 0
- joint arm_joint_2: limit lower=-1.57 upper=0 effort=1000.0 velocity=50.0 -> lower=0 upper=1.57 effort=1000.0 velocity=50.0; origin xyz=-0.072 0.0 -0.0568 rpy=0 1.57 0 -> xyz=-0.0568 0.0 0.072 rpy=0 1.57 0
- joint tool_joint: limit lower=-0.4 upper=0.8 effort=1000.0 velocity=50.0 -> lower=0.0 upper=1.57 effort=1000.0 velocity=50.0; origin xyz=0.09125 -0.00625 0.021 rpy=0 0 0 -> xyz=0.09125 -0.00625 0.021 rpy=0 0 -0.5
